Commit message: added rviz visualisation of urdf

File: ATV_models/UPDATED_polaris_ranger_xp900_no_roll_cage/model.urdf (robot description, URDF)
Before this commit: robot polaris_ranger_xp900, 12 links, 12 joints
Links:
- link polaris_ranger_xp900__brake_pedal: geometry collision box size=0.063 0.08 0.01; visual mesh filename=package://meshes/polaris.dae OR meshes/polaris.dae OR meshe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 scale=1.0 1.0 1.0
- link polaris_ranger_xp900__chassis: geometry collision box size=0.03 0.1 0.05; collision box size=0.03 0.1 0.1835
- link polaris_ranger_xp900__front_left_wheel: geometry collision cylinder length=0.2794 radius=0.3175; visual mesh filename=package://meshes/polaris.dae OR meshes/polaris.dae OR meshe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 scale=1.003700111 0.886200464 0.886200464
- link polaris_ranger_xp900__front_right_wheel: geometry collision cylinder length=0.2794 radius=0.3175; visual mesh filename=package://meshes/polaris.dae OR meshes/polaris.dae OR meshe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 scale=1.003700111 0.886200464 0.886200464
- link polaris_ranger_xp900__gas_pedal: geometry collision box size=0.1069000 0.0770000 0.010000; visual mesh filename=package://meshes/polaris.dae OR meshes/polaris.dae OR meshe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 scale=1.0 1.0 1.0
- link polaris_ranger_xp900__hand_brake: geometry collision mesh filename=package://meshes/polaris.dae OR meshes/polaris.dae OR meshe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 scale=1.0 1.0 1.0; visual mesh filename=package://meshes/polaris.dae OR meshes/polaris.dae OR meshe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 scale=1.0 1.0 1.0
- link polaris_ranger_xp900__rear_left_wheel: geometry collision cylinder length=0.2794 radius=0.3175; visual mesh filename=package://meshes/polaris.dae OR meshes/polaris.dae OR meshe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 scale=1.003700111 0.886200464 0.886200464
- link polaris_ranger_xp900__rear_right_wheel: geometry collision cylinder length=0.2794 radius=0.3175; visual mesh filename=package://meshes/polaris.dae OR meshes/polaris.dae OR meshe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 scale=1.003700111 0.886200464 0.886200464
- link polaris_ranger_xp900__steering_wheel: geometry collision mesh filename=package://meshes/polaris.dae OR meshes/polaris.dae OR meshe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 scale=1.0 1.0 1.0; visual mesh filename=package://meshes/polaris.dae OR meshes/polaris.dae OR meshe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 scale=1.0 1.0 1.0
Joints:
- removed joint polaris_ranger_xp900__rear_differential_joint
- joint polaris_ranger_xp900__FNR_switch_joint: type revolute -> fixed
- joint polaris_ranger_xp900__brake_joint: type prismatic -> fixed
- joint polaris_ranger_xp900__front_left_wheel_joint: type fixed -> continuous
- joint polaris_ranger_xp900__front_right_wheel_joint: type fixed -> continuous
- joint polaris_ranger_xp900__gas_joint: type prismatic -> fixed
- joint polaris_ranger_xp900__hand_brake_joint: type revolute -> fixed
- joint polaris_ranger_xp900__rear_left_wheel_joint: type fixed -> continuous
- joint polaris_ranger_xp900__rear_right_wheel_joint: type fixed -> continuous
- joint polaris_ranger_xp900__steering_joint: type revolute -> fixed
