Commit message: added hackerman controller but not working

File: ATV_ws/src/ATV_description/models/polaris_ranger_xp900_no_roll_cage/model copy.urdf (robot description, URDF)
Before this commit: robot polaris_ranger_xp900, 7 links, 6 joints
Links:
- removed link left_front_wheel
- removed link left_rear_wheel
- removed link right_front_wheel
- removed link right_rear_wheel
- added link fl_wheel, mass 12; collision cylinder length=0.2794 radius=0.3175; visual mesh filename=package://ATV_description/models/polaris_ranger_xp900_no_ro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 scale=1.0 1.0 1.0
- added link fr_wheel, mass 12; collision cylinder length=0.2794 radius=0.3175; visual mesh filename=package://ATV_description/models/polaris_ranger_xp900_no_ro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 scale=1.0 1.0 1.0
- added link rl_wheel, mass 12; collision cylinder length=0.2794 radius=0.3175; visual mesh filename=package://ATV_description/models/polaris_ranger_xp900_no_ro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 scale=1.0 1.0 1.0
- added link rr_wheel, mass 12; collision cylinder length=0.2794 radius=0.3175; visual mesh filename=package://ATV_description/models/polaris_ranger_xp900_no_ro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 scale=1.0 1.0 1.0
Joints:
- removed joint left_front_axle
- removed joint left_rear_axle
- removed joint left_steering_joint
- removed joint right_front_axle
- removed joint right_rear_axle
- removed joint right_steering_joint
- added joint fl_joint: type continuous, parent fl_steering_block, child fl_wheel, origin xyz=0      -0.00818 -0.21562 rpy=-3.09079  0       0, axis 0.00000000e+00   8.30000000e-04   1.00000000e+00, limit lower=0 upper=0 effort=0 velocity=0
- added joint fl_steering_joint: type revolute, parent chassis, child fl_steering_block, origin xyz=1.20222  0.5      0.35515 rpy=1.57079  0       0, axis 0  1  0, limit lower=-0.7727 upper=0.7727 effort=1000.0 velocity=1.0
- added joint fr_joint: type continuous, parent fr_steering_block, child fr_wheel, origin xyz=0      -0.00818  0.21562 rpy=-0.05079  0       0, axis 0.00000000e+00   8.30000000e-04  -1.00000000e+00, limit lower=0 upper=0 effort=0 velocity=0
- added joint fr_steering_joint: type revolute, parent chassis, child fr_steering_block, origin xyz=1.20222 -0.5      0.35515 rpy=1.57079  0       0, axis 0  1  0, limit lower=-0.7727 upper=0.7727 effort=1000.0 velocity=1.0
- added joint rl_joint: type continuous, parent chassis, child rl_wheel, origin xyz=-0.99377  0.71562  0.34697 rpy=-1.52  0    0, axis 0.00000000e+00   8.30000000e-04   1.00000000e+00, limit lower=100 upper=-100 effort=100 velocity=1
- added joint rr_joint: type continuous, parent chassis, child rr_wheel, origin xyz=-0.99377 -0.61574  0.34189 rpy=1.52  0    0, axis 0.00000000e+00   8.30000000e-04  -1.00000000e+00, limit lower=100 upper=-100 effort=100 velocity=1
