Commit message: solved URDF on Rviz

File: ATV_ws/src/ATV_description/models/polaris_ranger_xp900_no_roll_cage/model.urdf (robot description, URDF)
Before this commit: robot polaris_ranger_xp900, 12 links, 11 joints
Links:
- removed link polaris_ranger_xp900__FNR_switch
- removed link polaris_ranger_xp900__brake_pedal
- removed link polaris_ranger_xp900__gas_pedal
- removed link polaris_ranger_xp900__hand_brake
- removed link polaris_ranger_xp900__steering_wheel
- link polaris_ranger_xp900__chassis: geometry collision box size=0.03 0.1 0.05; collision box size=0.03 0.1 0.1835
- link polaris_ranger_xp900__front_left_wheel: geometry collision cylinder length=0.2794 radius=0.3175; visual mesh filename=package://ATV_description/models/polaris_ranger_xp900_no_ro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 scale=1.0 1.0 1.0
- link polaris_ranger_xp900__front_right_wheel: geometry collision cylinder length=0.2794 radius=0.3175; visual mesh filename=package://ATV_description/models/polaris_ranger_xp900_no_ro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 scale=1.0 1.0 1.0
- link polaris_ranger_xp900__rear_left_wheel: geometry collision cylinder length=0.2794 radius=0.3175; visual mesh filename=package://ATV_description/models/polaris_ranger_xp900_no_ro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 scale=1.0 1.0 1.0
- link polaris_ranger_xp900__rear_right_wheel: geometry collision cylinder length=0.2794 radius=0.3175; visual mesh filename=package://ATV_description/models/polaris_ranger_xp900_no_ro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 scale=1.0 1.0 1.0
Joints:
- removed joint polaris_ranger_xp900__FNR_switch_joint
- removed joint polaris_ranger_xp900__brake_joint
- removed joint polaris_ranger_xp900__gas_joint
- removed joint polaris_ranger_xp900__hand_brake_joint
- removed joint polaris_ranger_xp900__steering_joint

Commit message: started working on URDF actuators and transmissions

File: ATV_ws/src/ATV_description/models/polaris_ranger_xp900_no_roll_cage/model.urdf (robot description, URDF)
Before this commit: robot polaris_ranger_xp900, 7 links, 6 joints
Links:
- removed link polaris_ranger_xp900__chassis
- removed link polaris_ranger_xp900__front_left_wheel
- removed link polaris_ranger_xp900__front_left_wheel_steering_block
- removed link polaris_ranger_xp900__front_right_wheel
- removed link polaris_ranger_xp900__front_right_wheel_steering_block
- removed link polaris_ranger_xp900__rear_left_wheel
- removed link polaris_ranger_xp900__rear_right_wheel
- added link chassis, mass 720.0; collision box size=0.03 0.1 0.05; collision box size=0.03 0.1 0.1835
- added link fl_steering_block, mass 1; collision cylinder length=0.01 radius=0.05
- added link fl_wheel, mass 12; collision cylinder length=0.2794 radius=0.3175; visual mesh filename=package://ATV_description/models/polaris_ranger_xp900_no_ro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 scale=1.0 1.0 1.0
- added link fr_steering_block, mass 1; collision cylinder length=0.01 radius=0.05
- added link fr_wheel, mass 12; collision cylinder length=0.2794 radius=0.3175; visual mesh filename=package://ATV_description/models/polaris_ranger_xp900_no_ro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 scale=1.0 1.0 1.0
- added link rl_wheel, mass 12; collision cylinder length=0.2794 radius=0.3175; visual mesh filename=package://ATV_description/models/polaris_ranger_xp900_no_ro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 scale=1.0 1.0 1.0
- added link rr_wheel, mass 12; collision cylinder length=0.2794 radius=0.3175; visual mesh filename=package://ATV_description/models/polaris_ranger_xp900_no_ro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 scale=1.0 1.0 1.0
Joints:
- removed joint polaris_ranger_xp900__front_left_steering_joint
- removed joint polaris_ranger_xp900__front_left_wheel_joint
- removed joint polaris_ranger_xp900__front_right_steering_joint
- removed joint polaris_ranger_xp900__front_right_wheel_joint
- removed joint polaris_ranger_xp900__rear_left_wheel_joint
- removed joint polaris_ranger_xp900__rear_right_wheel_joint
- added joint fl_joint: type continuous, parent fl_steering_block, child fl_wheel, origin xyz=0      -0.00818 -0.21562 rpy=-3.09079  0       0, axis 0.00000000e+00   8.30000000e-04   1.00000000e+00, limit lower=0 upper=0 effort=0 velocity=0
- added joint fl_steering_joint: type revolute, parent chassis, child fl_steering_block, origin xyz=1.20222  0.5      0.35515 rpy=1.57079  0       0, axis 0  1  0, limit lower=-0.7727 upper=0.7727 effort=0.0 velocity=0.0
- added joint fr_joint: type continuous, parent fr_steering_block, child fr_wheel, origin xyz=0      -0.00818  0.21562 rpy=-0.05079  0       0, axis 0.00000000e+00   8.30000000e-04  -1.00000000e+00, limit lower=0 upper=0 effort=0 velocity=0
- added joint fr_steering_joint: type revolute, parent chassis, child fr_steering_block, origin xyz=1.20222 -0.5      0.35515 rpy=1.57079  0       0, axis 0  1  0, limit lower=-0.7727 upper=0.7727 effort=0.0 velocity=0.0
- added joint rl_joint: type continuous, parent chassis, child rl_wheel, origin xyz=-0.99377  0.71562  0.34697 rpy=-1.52  0    0, axis 0.00000000e+00   8.30000000e-04   1.00000000e+00, limit lower=0 upper=0 effort=0 velocity=0
- added joint rr_joint: type continuous, parent chassis, child rr_wheel, origin xyz=-0.99377 -0.61574  0.34189 rpy=1.52  0    0, axis 0.00000000e+00   8.30000000e-04  -1.00000000e+00, limit lower=0 upper=0 effort=0 velocity=0

Commit message: woking topics for control pkg

File: ATV_ws/src/ATV_description/models/polaris_ranger_xp900_no_roll_cage/model.urdf (robot description, URDF)
Before this commit: robot polaris_ranger_xp900, 7 links, 6 joints
Joints:
- joint fl_steering_joint: limit lower=-0.7727 upper=0.7727 effort=0.0 velocity=0.0 -> lower=-0.7727 upper=0.7727 effort=1000.0 velocity=1.0
- joint fr_steering_joint: limit lower=-0.7727 upper=0.7727 effort=0.0 velocity=0.0 -> lower=-0.7727 upper=0.7727 effort=1000.0 velocity=1.0
- joint rl_joint: limit lower=0 upper=0 effort=0 velocity=0 -> lower=100 upper=-100 effort=100 velocity=1
- joint rr_joint: limit lower=0 upper=0 effort=0 velocity=0 -> lower=100 upper=-100 effort=100 velocity=1

Commit message: now keyboard control works decently

File: ATV_ws/src/ATV_description/models/polaris_ranger_xp900_no_roll_cage/model.urdf (robot description, URDF)
Before this commit: robot polaris_ranger_xp900, 7 links, 6 joints
Joints:
- joint left_rear_axle: limit lower=100 upper=-100 effort=100 velocity=1 -> lower=-100 upper=100 effort=100 velocity=100.0
- joint right_rear_axle: limit lower=100 upper=-100 effort=100 velocity=1 -> lower=-100 upper=100 effort=100 velocity=100.0

Commit message: zioporco c'è un joint state pub che salta fuori a caso

File: ATV_ws/src/ATV_description/models/polaris_ranger_xp900_no_roll_cage/model.urdf (robot description, URDF)
Before this commit: robot polaris_ranger_xp900, 7 links, 6 joints
Links:
- added link base_link
Joints:
- added joint base_joint: type fixed, parent base_link, child chassis
