Commit message: added IMU, lidar, Kinect MILESTON ----

File: ATV_ws/src/ATV_description/models/polaris_ranger_xp900_no_roll_cage/model2.urdf (robot description, URDF)
Before this commit: robot polaris_ranger_xp900, 8 links, 7 joints
Links:
- added link imu_frame; collision box size=0.06 0.06 0.03; visual box size=0.06 0.06 0.03
- added link kinect_frame; collision box size=0.06 0.06 0.03; visual box size=0.03 0.07 0.03
- added link laser_frame; collision cylinder length=0.04 radius=0.05; visual cylinder length=0.04 radius=0.05
Joints:
- added joint imu_joint: type fixed, parent chassis, child imu_frame, origin xyz=0.1 0 0.9 rpy=0 0 0
- added joint kinect_joint: type fixed, parent chassis, child kinect_frame, origin xyz=1.3 0 1 rpy=0 0 0
- added joint laser_joint: type fixed, parent chassis, child laser_frame, origin xyz=1.3 0 0.9 rpy=0 0 0

Commit message: added gps and driver pov, last commit before hard reset

File: ATV_ws/src/ATV_description/models/polaris_ranger_xp900_no_roll_cage/model2.urdf (robot description, URDF)
Before this commit: robot polaris_ranger_xp900, 11 links, 10 joints
Links:
- removed link kinect_frame
- added link camera_link, mass 1e-5; visual box size=0.3 0.3 0.3
- added link gps_link, mass 1; collision box size=0.1 0.1 0.1; visual box size=0.1 0.1 0.1
- added link kinect_frame_optical
- added link kinect_link; collision box size=0.07 0.3 0.09; visual box size=0.07 0.3 0.09
- link chassis: geometry collision box size=0.03 0.1 0.05; collision box size=0.03 0.1 0.1835
Joints:
- removed joint kinect_joint
- removed joint laser_joint
- added joint camera_joint: type fixed, parent chassis, child camera_link, origin xyz=0 0.3 1.6 rpy=0 0 0, axis 0 1 0
- added joint gps_joint: type fixed, parent chassis, child gps_link
- added joint kinect_frame_joint: type fixed, parent chassis, child kinect_link, origin xyz=1.3 0 1 rpy=0 0 0
- added joint kinect_optical_joint: type fixed, parent kinect_link, child kinect_frame_optical, origin xyz=0 0 0 rpy=-1.5708 0 -1.5708
- added joint sensorr_joint: type fixed, parent chassis, child laser_frame, origin xyz=1.3 0 0.7 rpy=0 0 0
